File: nucleo144 and 3.2 ILI9341 lcd parallel 16bit/nucleo144 and 3.2 ILI9341 lcd parallel 16bit.kicad_pcb (KiCad board)
At the start: 2 copper layers, 100 x 70 mm, 6 parts, among them U1 NUCLEO144

Commit message: Signed-off-by: DamianPodrazaCode <damian.podraza@gmail.com>
Routing:
- net GND: vias 0 -> 7
Changed lines of the file:
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@@
   (segment (start 201.374 102.521) (end 157.631 102.521) (width 0.4) (layer "B.Cu") (net 99))
   (segment (start 157.631 102.521) (end 157.448 102.338) (width 0.4) (layer "B.Cu") (net 99))
+  (via (at 121.666 108.966) (size 1.5) (drill 0.4) (layers "F.Cu" "B.Cu") (free) (net 105))
+  (via (at 155.448 81.28) (size 1.5) (drill 0.4) (layers "F.Cu" "B.Cu") (free) (net 105))
+  (via (at 121.92 81.026) (size 1.5) (drill 0.4) (layers "F.Cu" "B.Cu") (free) (net 105))
+  (via (at 190.5 106.934) (size 1.5) (drill 0.4) (layers "F.Cu" "B.Cu") (free) (net 105))
+  (via (at 146.812 107.188) (size 1.5) (drill 0.4) (layers "F.Cu" "B.Cu") (free) (net 105))
+  (via (at 146.812 81.28) (size 1.5) (drill 0.4) (layers "F.Cu" "B.Cu") (free) (net 105))
+  (via (at 134.874 81.28) (size 1.5) (drill 0.4) (layers "F.Cu" "B.Cu") (free) (net 105))
   (segment (start 203.914 105.061) (end 201.374 107.601) (width 0.4) (layer "B.Cu") (net 105))
   (segment (start 130.804 109.932) (end 130.804 65.663) (width 0.4) (layer "F.Cu") (net 107))
