File: nucleo144 and 3.2 ILI9341 lcd parallel 16bit/nucleo144 and 3.2 ILI9341 lcd parallel 16bit.kicad_sch (KiCad schematic)
At the start: 2 parts, among them U1 NUCLEO144

Commit message: Signed-off-by: DamianPodrazaCode <damian.podraza@gmail.com>
Connections:
- no-connect marks 0 -> 97
Other:
- moved on the sheet: TFT1
