File: nucleo144 and 2.2 S6D0164 lcd parallel 16bit/nucleo144 and 2.2 S6D0164 lcd parallel 16bit.kicad_pcb (KiCad board)
At the start: 2 copper layers, 100 x 70 mm, 6 parts, among them U1 NUCLEO144

Commit message: Signed-off-by: DamianPodrazaCode <damian.podraza@gmail.com>
Parts:
- added SW1: SW_Push, Button_Switch_THT:SW_PUSH_6mm, F.Cu at (123.3, 110.6)
- added SW2: SW_Push, Button_Switch_THT:SW_PUSH_6mm, F.Cu at (113.7, 102.9)
- added SW3: SW_Push, Button_Switch_THT:SW_PUSH_6mm, F.Cu at (132.9, 103.0)
- added SW4: SW_Push, Button_Switch_THT:SW_PUSH_6mm, F.Cu at (123.3, 95.3)
- added SW5: SW_Push, Button_Switch_THT:SW_PUSH_6mm, F.Cu at (114.1, 78.5)
- added SW6: SW_Push, Button_Switch_THT:SW_PUSH_6mm, F.Cu at (124.9, 78.4)
Connections:
- U1 pad 1: unconnected-(U1-PC10-Pad1) -> sw1
- U1 pad 2: unconnected-(U1-PC11-Pad2) -> sw2
- U1 pad 3: unconnected-(U1-PC12-Pad3) -> sw3
- U1 pad 4: unconnected-(U1-PD2-Pad4) -> sw4
- U1 pad 75: unconnected-(U1-PB8-Pad75) -> sw5
- U1 pad 77: unconnected-(U1-PB9-Pad77) -> sw6
Routing:
- net sw4: track 0.00 -> 39.2 mm
- net sw3: track 0.00 -> 36.2 mm
- net sw2: track 0.00 -> 32.2 mm
- net sw1: track 0.00 -> 25.7 mm
- net sw6: track 0.00 -> 21.0 mm
- net sw5: track 0.00 -> 20.4 mm
- net D13: track 100.3 -> 88.9 mm
- net SPI_MISO: track 81.6 -> 76.4 mm
- net SPI_CLK: track 81.7 -> 76.9 mm
