File: nucleo144 and 2.2 ILI9341 lcd SPI/nucleo144 and 2.2 ILI9341 lcd SPI.kicad_sch (KiCad schematic)
At the start: 5 parts, among them U1 NUCLEO144, U2 AMS1117-3.3

Commit message: Signed-off-by: DamianPodrazaCode <damian.podraza@gmail.com>
Parts:
- removed C1, C2: C_Polarized, Capacitor_Tantalum_SMD:CP_EIA-3528-12_Kemet-T, symbol Device:C_Polarized
- removed TFT1: 4.3 TFT SSD1963 parallel, zombie_display:4.3_TFT_SSD1963, symbol zombie_display:4.3_TFT_SDD1963
- removed U2: AMS1117-3.3, Package_TO_SOT_SMD:SOT-223-3_TabPin2, symbol Regulator_Linear:AMS1117-3.3
- added SW1, SW2, SW3, SW4, SW5, SW6: SW_Push, Button_Switch_THT:SW_PUSH_6mm, symbol Switch:SW_Push
- added TFT1: 2.2_TFT_ILI9341_SPI, zombie_display:2.2_TFT_ILI9341_SPI, symbol zombie_display:2.2_TFT_ILI9341_SPI
Connections:
- net 5V: now also TFT1.1 (VCC)
- net GND: now also SW1.2, SW2.2, SW3.2, SW4.2, SW5.2, SW6.2, TFT1.2 (GND)
- net LCD_BL: now also TFT1.8 (LED)
- net LCD_CS: now also TFT1.3 (CS)
- net LCD_RS: now also TFT1.5 (D/C)
- net LCD_RST: now also TFT1.4 (RESET)
- net SD_CLK: now also TFT1.13 (SD_SCK)
- net SD_CS: now also TFT1.10 (SD_CS)
- net SD_MISO: now also TFT1.12 (SD_MISO)
- net SD_MOSI: now also TFT1.11 (SD_MOSI)
- net SPI_CLK: now also TFT1.7 (SCK)
- net SPI_MISO: now also TFT1.9 (MISO)
- net SPI_MOSI: now also TFT1.6 (MOSI)
- net sw6: now reaches U1.133 (PG14)
- net sw6: now also SW6.1
- net sw2: now reaches U1.138 (PG8)
- net sw2: now also SW2.1
- net sw1: now reaches U1.140 (PG5)
- net sw1: now also SW1.1
- net sw3: now reaches U1.63 (PG9)
- net sw3: now also SW3.1
- net sw5: now reaches U1.65 (PG12)
- net sw5: now also SW5.1
- net sw4: now reaches U1.66 (PG10)
- net sw4: now also SW4.1

Commit message: Signed-off-by: DamianPodrazaCode <damian.podraza@gmail.com>
Connections:
- net D0: no longer names the net of U1.118 (PD14)
- net D1: no longer names the net of U1.120 (PD15)
- net D10: no longer names the net of U1.127 (PE13)
- net D11: no longer names the net of U1.123 (PE14)
- net D12: no longer names the net of U1.125 (PE15)
- net D13: no longer names the net of U1.82 (STLINK_TX/PD8)
- net D14: no longer names the net of U1.69 (STLINK_RX/PD9)
- net D15: no longer names the net of U1.137 (PD10)
- net D2: no longer names the net of U1.57 (PD0)
- net D3: no longer names the net of U1.55 (PD1)
- net D4: no longer names the net of U1.116 (PE7)
- net D5: no longer names the net of U1.112 (PE8)
- net D6: no longer names the net of U1.124 (PE9)
- net D7: no longer names the net of U1.119 (PE10)
- net D8: no longer names the net of U1.128 (PE11)
- net D9: no longer names the net of U1.121 (PE12)
- net F_CS: no longer names the net of U1.96 (PB1)
- net LCD_RD: no longer names the net of U1.39 (PD4)
- net LCD_WR: no longer names the net of U1.41 (PD5)
- net PEN: no longer names the net of U1.37 (PC3)
- net T_CS: no longer names the net of U1.109 (PA3)
- no-connect marks 0 -> 108
