File: nucleo144 and 2.2 ILI9341 lcd SPI/nucleo144 and 2.2 ILI9341 lcd SPI.kicad_pcb (KiCad board)
At the start: 2 copper layers, 100 x 70 mm, 12 parts, among them SW1 SW_Push, SW2 SW_Push, SW3 SW_Push, SW4 SW_Push, SW5 SW_Push, SW6 SW_Push, U1 NUCLEO144

Commit message: Signed-off-by: DamianPodrazaCode <damian.podraza@gmail.com>
Routing:
- net SD_CS: track 76.1 -> 0.00 mm, vias 1 -> 0
- net SD_CLK: track 40.1 -> 0.00 mm, vias 1 -> 0
- net SD_MISO: track 39.8 -> 0.00 mm, vias 1 -> 0
- net SD_MOSI: track 32.5 -> 0.00 mm, vias 1 -> 0
- removed copper zone on B.Cu, net (none)
Changed lines of the file:
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@@
     )
   )
-  (gr_rect (start 214.3 130.048) (end 114.3 60.048)
+  (gr_rect (start 114.3 60.048) (end 214.3 130.048)
     (stroke (width 0.1) (type default)) (fill none) (layer "Edge.Cuts"))
-  (segment (start 117.094 61.0616) (end 144.7292 61.0616) (width 0.4) (layer "F.Cu") (net 109))
-  (segment (start 144.7292 61.0616) (end 145.3 61.6324) (width 0.4) (layer "F.Cu") (net 109))
-  (segment (start 118.1608 102.108) (end 115.7732 99.7204) (width 0.4) (layer "F.Cu") (net 109))
-  (segment (start 145.3 61.6324) (end 145.3 63.308) (width 0.4) (layer "F.Cu") (net 109))
-  (segment (start 115.7732 62.3824) (end 117.094 61.0616) (width 0.4) (layer "F.Cu") (net 109))
-  (segment (start 115.7732 99.7204) (end 115.7732 62.3824) (width 0.4) (layer "F.Cu") (net 109))
-  (via (at 118.1608 102.108) (size 1.5) (drill 0.4) (layers "F.Cu" "B.Cu") (net 109))
-  (segment (start 118.165 98.663) (end 118.165 102.1038) (width 0.4) (layer "B.Cu") (net 109))
-  (segment (start 118.165 102.1038) (end 118.1608 102.108) (width 0.4) (layer "B.Cu") (net 109))
-  (segment (start 121.19 116.618) (end 121.19 125.558) (width 0.4) (layer "F.Cu") (net 128))
-  (segment (start 121.19 125.558) (end 122.44 126.808) (width 0.4) (layer "F.Cu") (net 128))
-  (segment (start 121.0564 116.4844) (end 121.19 116.618) (width 0.4) (layer "F.Cu") (net 128))
-  (via (at 121.0564 116.4844) (size 1.5) (drill 0.4) (layers "F.Cu" "B.Cu") (net 128))
-  (segment (start 118.165 96.123) (end 121.0564 99.0144) (width 0.4) (layer "B.Cu") (net 128))
-  (segment (start 121.0564 99.0144) (end 121.0564 116.4844) (width 0.4) (layer "B.Cu") (net 128))
-  (segment (start 116.0272 125.2728) (end 117.5624 126.808) (width 0.4) (layer "F.Cu") (net 129))
-  (segment (start 117.5624 126.808) (end 119.9 126.808) (width 0.4) (layer "F.Cu") (net 129))
-  (via (at 116.0272 125.2728) (size 1.5) (drill 0.4) (layers "F.Cu" "B.Cu") (net 129))
-  (segment (start 118.165 91.043) (end 115.4684 93.7396) (width 0.4) (layer "B.Cu") (net 129))
-  (segment (start 115.4684 93.7396) (end 115.4684 124.714) (width 0.4) (layer "B.Cu") (net 129))
-  (segment (start 115.4684 124.714) (end 116.0272 125.2728) (width 0.4) (layer "B.Cu") (net 129))
-  (segment (start 117.5004 123.7996) (end 119.4316 123.7996) (width 0.4) (layer "F.Cu") (net 130))
-  (segment (start 119.4316 123.7996) (end 119.9 124.268) (width 0.4) (layer "F.Cu") (net 130))
-  (via (at 117.5004 123.7996) (size 1.5) (drill 0.4) (layers "F.Cu" "B.Cu") (net 130))
-  (segment (start 118.618 122.2756) (end 117.5004 123.3932) (width 0.4) (layer "B.Cu") (net 130))
-  (segment (start 123.0376 96.4692) (end 123.0376 120.3452) (width 0.4) (layer "B.Cu") (net 130))
-  (segment (start 120.1514 93.583) (end 123.0376 96.4692) (width 0.4) (layer "B.Cu") (net 130))
-  (segment (start 121.2088 122.2756) (end 118.618 122.2756) (width 0.4) (layer "B.Cu") (net 130))
-  (segment (start 117.5004 123.3932) (end 117.5004 123.7996) (width 0.4) (layer "B.Cu") (net 130))
-  (segment (start 118.165 93.583) (end 120.1514 93.583) (width 0.4) (layer "B.Cu") (net 130))
-  (segment (start 123.0884 120.396) (end 121.2088 122.2756) (width 0.4) (layer "B.Cu") (net 130))
-  (segment (start 123.0376 120.3452) (end 123.0884 120.396) (width 0.4) (layer "B.Cu") (net 130))
   (zone (net 102) (net_name "GND") (layers "F&B.Cu") (hatch edge 0.5)
     (connect_pads (clearance 0.5))
@@
       )
     )
-  )
-  (zone (net 0) (net_name "") (layer "B.Cu") (hatch edge 0.5)
-    (priority 1)
-    (connect_pads (clearance 0.5))
-    (min_thickness 0.25) (filled_areas_thickness no)
-    (fill yes (thermal_gap 0.5) (thermal_bridge_width 0.5))
-    (polygon
-      (pts
-        (xy 161 78)
-        (xy 161 82)
-        (xy 191 82)
-        (xy 191 78)
-      )
-    )

Commit message: Signed-off-by: DamianPodrazaCode <damian.podraza@gmail.com>
Parts:
- moved SW3 29.7 mm to (196.2, 110.2), turned to 180 degrees
- moved SW6 28.4 mm to (186.7, 82.1)
- moved SW5 19.9 mm to (209.0, 110.3), turned to 180 degrees
- moved SW2 12.7 mm to (196.2, 73.6)
- moved SW1 12.5 mm to (205.5, 82.0)
- moved SW4 7.90 mm to (202.6, 94.8), turned to 180 degrees
Routing:
- net SPI_CLK: track 0.00 -> 72.9 mm, vias 0 -> 1
- net SPI_MISO: track 0.00 -> 65.1 mm, vias 0 -> 1
- net SD_CS: track 0.00 -> 64.3 mm, vias 0 -> 1
- net 5V: track 0.00 -> 60.6 mm, vias 0 -> 1
- net LCD_BL: track 0.00 -> 60.0 mm, vias 0 -> 1
- net SPI_MOSI: track 0.00 -> 52.2 mm, vias 0 -> 1
- net LCD_RST: track 0.00 -> 42.6 mm, vias 0 -> 1
- net SD_CLK: track 0.00 -> 41.4 mm, vias 0 -> 1
- net sw4: track 0.00 -> 36.7 mm, vias 0 -> 1
- net SD_MOSI: track 0.00 -> 36.6 mm, vias 0 -> 1
- net LCD_RS: track 0.00 -> 34.5 mm, vias 0 -> 1
- net LCD_CS: track 0.00 -> 34.4 mm, vias 0 -> 1
- net SD_MISO: track 0.00 -> 33.9 mm, vias 0 -> 1
- net sw1: track 0.00 -> 25.9 mm, vias 0 -> 1
- net sw3: track 0.00 -> 24.1 mm, vias 0 -> 1
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