File: nucleo144 and 4.3 SSD1963 lcd parallel 16bit/nucleo144 and 4.3 SSD1963 lcd parallel 16bit.kicad_sch (KiCad schematic)
At the start: 5 parts, among them U1 NUCLEO144, U2 AMS1117-3.3

Commit message: Signed-off-by: DamianPodrazaCode <damian.podraza@gmail.com>
Connections:
- no-connect marks 0 -> 99
